File: TPS5420.kicad_pcb (KiCad board)
At the start: 2 copper layers, 46.3 x 18.1 mm, 12 parts, among them J1 Screw_Terminal_01x02, J2 Screw_Terminal_01x02, U1 TPS5420D, U2 CDBC560-G

Commit message: SHifted out capacitors
Parts:
- moved C3 6.32 mm to (150.5, 90.5)
- moved C4 6.32 mm to (150.5, 93.3)
- moved C5 6.32 mm to (150.4, 96.3)
- moved J2 5.61 mm to (149.3, 83.6), turned to 0 degrees
- moved R1 3.43 mm to (143.5, 80.0), turned to 0 degrees
- moved C1 2.83 mm to (129.2, 83.8), turned to -90 degrees
- moved L1 1.86 mm to (140.9, 91.6)
- moved U2 1.74 mm to (131.8, 91.6), turned to 180 degrees
- moved J1 1.09 mm to (120.5, 90.2)
- moved R2 1.07 mm to (143.5, 83.1), turned to 180 degrees
- moved C2 0.69 mm to (140.0, 86.8)
Connections:
- J2 pad 1: GND -> /Vout
- J2 pad 2: /Vout -> GND
Routing:
- net Net-(U1-PH): track 20.9 -> 15.9 mm
- net /Vout: track 27.6 -> 25.1 mm
- net GND: track 6.87 -> 9.23 mm, vias 33 -> 38
- net Net-(U1-VSENSE): track 7.60 -> 6.68 mm
Other:
- board size 46.3 x 18.1 mm -> 46.3 x 21.1 mm
